File: KiCAD/TMi-3/TMi-3.kicad_pcb (KiCad board)
At the start: 2 copper layers, 50 x 155.5 mm, 40 parts, among them J1 MJ-3536NG, J10 NMJ4HFD3, J2 MJ-3536NG, J3 Power_Screw_Terminal, J4 MJ-3536NG, J5 MJ-3536NG, J7 NMJ4HFD3, J8 NMJ4HFD3, J9 NMJ4HFD3, Q1 IRLZ44N, Q2 IRLZ44N, Q3 IRLZ44N, Q4 IRLZ44N

Commit message: Journal Entries
Parts:
- removed the J3 at (48.9, 38.5)
- added H3: MountingHole_Pad, MountingHole:MountingHole_2.2mm_M2_DIN965_Pad_TopBottom, F.Cu at (101.5, 166.5)
- added J9: Barrel_Jack_Switch, Connector_BarrelJack:BarrelJack_Horizontal, F.Cu at (40.5, 41.5)
- C9: footprint Capacitor_THT:CP_Radial_D10.0mm_P5.00mm -> PCM_Capacitor_THT_AKL:CP_Radial_D10.0mm_P5.00mm_H20mm_Horizontal1_Supported
- J1, J2: footprint MJ:MJ3536NG -> Connector_Audio:MJ3536NG_Tighter_Pads
- J3: renamed from J4; footprint MJ:MJ3536NG -> Connector_Audio:MJ3536NG_Tighter_Pads
- J4: renamed from J5; footprint MJ:MJ3536NG -> Connector_Audio:MJ3536NG_Tighter_Pads
- moved H1 59.6 mm to (92.5, 41.5)
- moved H2 51.9 mm to (102.5, 139.5)
- moved C9 16.1 mm to (50.1, 44.0), turned to 90 degrees
- moved R4 7.81 mm to (67.5, 93.0)
- moved R6 7.81 mm to (67.5, 128.0)
- moved R8 7.81 mm to (67.5, 163.5)
- moved C1 7.81 mm to (63.5, 76.5)
- moved C2 7.81 mm to (55.5, 74.3)
- moved C3 7.81 mm to (63.0, 111.5)
- moved C4 7.81 mm to (55.5, 109.4)
- moved C5 7.81 mm to (63.0, 146.3)
- moved C6 7.81 mm to (55.5, 144.4)
- moved C7 7.81 mm to (62.5, 182.0)
- moved C8 7.81 mm to (55.5, 179.9)
- moved D1 7.81 mm to (61.9, 51.0)
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- renumbered J7 to J5, J8 to J6, J9 to J7, J10 to J8
Connections:
- J1 pad 2: unconnected-(J1-Pad2) -> +12V
- J2 pad 2: unconnected-(J2-Pad2) -> +12V
- J3 pad 2: unconnected-(J4-Pad2) -> +12V
- J4 pad 2: unconnected-(J5-Pad2) -> +12V
Routing:
- net +12V: track 333.7 -> 371.7 mm
- net Net-(J7-PadT): track 14.6 -> 18.3 mm
- net Net-(J6-PadT): track 14.6 -> 18.2 mm
- net Net-(J8-PadT): track 14.6 -> 18.2 mm
- net Net-(J5-PadT): track 14.6 -> 18.1 mm
Other:
- board size 50 x 155.5 mm -> 50 x 160 mm
