File: KiCAD/TMi-3/TMi-3.kicad_sch (KiCad schematic)
At the start: 40 parts, among them J1 MJ-3536NG, J10 NMJ4HFD3, J2 MJ-3536NG, J3 Power_Screw_Terminal, J4 MJ-3536NG, J5 MJ-3536NG, J7 NMJ4HFD3, J8 NMJ4HFD3, J9 NMJ4HFD3, Q1 IRLZ44N, Q2 IRLZ44N, Q3 IRLZ44N, Q4 IRLZ44N

Commit message: Journal Entries
Parts:
- removed J3: Power_Screw_Terminal, TerminalBlock_RND:TerminalBlock_RND_205-00045_1x02_P5.00mm_Horizontal, symbol Connector:Screw_Terminal_01x02
- added H3: MountingHole_Pad, MountingHole:MountingHole_2.2mm_M2_DIN965_Pad_TopBottom, symbol Mechanical:MountingHole_Pad
- added J9: Barrel_Jack_Switch, Connector_BarrelJack:BarrelJack_Horizontal, symbol Connector:Barrel_Jack_Switch
- J1, J2: footprint MJ:MJ3536NG -> Connector_Audio:MJ3536NG_Tighter_Pads
- J3: renamed from J4; footprint MJ:MJ3536NG -> Connector_Audio:MJ3536NG_Tighter_Pads
- J4: renamed from J5; footprint MJ:MJ3536NG -> Connector_Audio:MJ3536NG_Tighter_Pads
- renumbered J7 to J5, J8 to J6, J9 to J7, J10 to J8
Connections:
- net +12V: now also J1.2, J2.2, J3.2, J4.2, J9.1
- net GND: now also J9.2
- no-connect marks 14 -> 12
